File: infinite_keyboard/infinite_keyboard.kicad_pcb (KiCad board)
At the start: 2 copper layers, 109 parts, among them IC1 ESP32-S3-WROOM-1-N8, IC2 MIC5504-3.3YM5-TR, IC3 PCM5100APWR, IC4 TPA6130A2RTJR, J1 UJ20-C-H-G-SMT-5-P16-TR, J2 MSD-1-A, J3 SJ-43617-SMT-TR

Commit message: Lots of updates
Parts:
- removed IC2: MIC5504-3.3YM5-TR, libraries:SOT95P280X145-5N
- added IC5: AP2112K-3.3TRG1, libraries:SOT95P285X140-5N, B.Cu at (303.2, 46.9)
- added R20: 22, Resistor_SMD:R_0805_2012Metric, B.Cu at (226.3, 74.5)
- added R21: 22, Resistor_SMD:R_0805_2012Metric, B.Cu at (224.2, 74.5)
- added R22: 22, Resistor_SMD:R_0805_2012Metric, B.Cu at (222.2, 74.5)
- added R23: 10k, Resistor_SMD:R_0805_2012Metric, B.Cu at (147.1, 63.8)
- added R24: 22, Resistor_SMD:R_0805_2012Metric, B.Cu at (220.2, 74.5)
- added R25: 10k, Resistor_SMD:R_0805_2012Metric, B.Cu at (153.8, 63.8)
- added R26: 10k, Resistor_SMD:R_0805_2012Metric, B.Cu at (145.0, 63.8)
- C24, C3: value C -> 1uF
- IC1: moved to B.Cu
- J3: moved to F.Cu
- moved BOOT1 292.7 mm to (-9.43, 52.2)
- moved RESET1 292.7 mm to (-9.43, 60.1)
- moved C1 279.4 mm to (-5.92, 59.7)
- moved R1 279.4 mm to (-5.89, 61.8)
- moved C3 279.3 mm to (-5.90, 51.8), turned to 180 degrees
- moved R2 279.3 mm to (-5.88, 53.9), turned to 180 degrees
- moved MODE_B1 245.9 mm to (264.9, 47.1)
- moved R17 237.7 mm to (266.8, 49.1), turned to 0 degrees
- moved MODE_A1 237.0 mm to (256.4, 47.2)
- moved R15 231.4 mm to (258.3, 49.1), turned to 0 degrees
- moved RUNNING1 228.0 mm to (247.7, 47.2)
- moved POWER1 219.5 mm to (239.4, 47.3)
- moved R14 216.1 mm to (249.6, 49.2), turned to 0 degrees
- moved R16 214.7 mm to (241.3, 49.3), turned to 0 degrees
- moved R12 80.9 mm to (147.3, 56.4), turned to 90 degrees
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Connections:
- C26 pad 1: +3.3V -> GND
- C3 pad 1: +3.3V -> GND
- IC1 pad 10: ROW3 -> LRCK
- IC1 pad 11: ROW4 -> DIN
- IC1 pad 12: ROW5 -> BCK
- IC1 pad 15: ROW6 -> Net-(IC1-IO3)
- IC1 pad 16: Net-(IC1-IO46) -> unconnected-(IC1-IO46-Pad16)
- IC1 pad 30: TPA_SCL -> COL1
- IC1 pad 31: TPA_SDA -> COL2
- IC1 pad 32: Net-(IC1-IO39) -> COL3
- IC1 pad 33: Net-(IC1-IO40) -> COL4
- IC1 pad 34: Net-(IC1-IO41) -> ROW1
- IC1 pad 35: Net-(IC1-IO42) -> ROW2
- IC1 pad 36: unconnected-(IC1-RXD0-Pad36) -> ROW3
- IC1 pad 37: unconnected-(IC1-TXD0-Pad37) -> ROW4
- IC1 pad 38: unconnected-(IC1-IO2-Pad38) -> ROW5
- IC1 pad 39: unconnected-(IC1-IO1-Pad39) -> ROW6
- IC1 pad 4: COL1 -> unconnected-(IC1-IO4-Pad4)
- IC1 pad 5: COL2 -> unconnected-(IC1-IO5-Pad5)
- IC1 pad 6: COL3 -> unconnected-(IC1-IO6-Pad6)
- IC1 pad 7: COL4 -> TPA_SCL
- IC1 pad 8: ROW1 -> TPA_SDA
- IC1 pad 9: ROW2 -> XSMT
- IC3 pad 13: Net-(IC1-IO39) -> BCK
- IC3 pad 14: Net-(IC1-IO40) -> DIN
- IC3 pad 15: Net-(IC1-IO41) -> LRCK
- IC3 pad 17: Net-(IC1-IO42) -> XSMT
- J2 pad 1: unconnected-(J2-DAT2-Pad1) -> Net-(J2-DAT2)
- J2 pad 2: Net-(IC1-IO48) -> Net-(J2-CD/DAT3)
- J2 pad 3: Net-(IC1-IO47) -> Net-(J2-CMD)
- J2 pad 5: Net-(IC1-IO21) -> Net-(J2-CLK)
- J2 pad 7: Net-(IC1-IO14) -> Net-(J2-DAT0)
- J2 pad 8: unconnected-(J2-DAT1-Pad8) -> Net-(J2-DAT1)
- J3 pad 4: unconnected-(J3-RING_2-Pad4) -> GND
- MODE_B1 pad 1: Net-(IC1-IO46) -> Net-(IC1-IO3)
- R10 pad 1: Net-(IC1-IO48) -> Net-(J2-DAT0)
- R11 pad 1: Net-(IC1-IO47) -> Net-(J2-CLK)
- R12 pad 1: Net-(IC1-IO21) -> Net-(J2-CMD)
- R13 pad 1: Net-(IC1-IO14) -> Net-(IC5-EN)
- R13 pad 2: +3.3V -> +5V
- RESET1 pad 1: unconnected-(RESET1-Pad1) -> GND
- RESET1 pad 2: unconnected-(RESET1-Pad2) -> Net-(IC1-EN)
Routing:
- net +3.3V: track 18.0 -> 0.00 mm
- net Net-(IC4-HPRIGHT): track 15.5 -> 0.00 mm
- net USB_DN: track 13.0 -> 0.00 mm, vias 2 -> 0
- net Net-(IC3-OUTR): track 12.0 -> 0.00 mm
- net Net-(IC4-HPLEFT): track 11.7 -> 0.00 mm, vias 2 -> 0
- net Net-(IC3-OUTL): track 9.40 -> 0.00 mm
- net USB_DP: track 9.24 -> 0.00 mm
- net Net-(J1-CC1): track 6.53 -> 0.00 mm, vias 1 -> 0
- net Net-(J1-CC2): track 6.28 -> 0.00 mm, vias 1 -> 0
- net Net-(C15-Pad1): track 6.16 -> 0.00 mm
- net Net-(IC3-LDOO): track 5.27 -> 0.00 mm
- net TPA_SCL: track 5.07 -> 0.00 mm
- net Net-(IC3-CAPP): track 4.71 -> 0.00 mm
- net Net-(C14-Pad2): track 4.42 -> 0.00 mm
- net Net-(IC4-CPVSS_1): track 4.05 -> 0.00 mm
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Other:
- board outline added: 293 x 49.5 mm

Commit message: Misc changes
Parts:
- BOOT1, MODE_A2, MODE_B2, RESET1: value SW_Push_Dual -> TS04-66-75-BK-160-SMT; footprint Button_Switch_THT:SW_PUSH_6mm_H4.3mm -> libraries:TS046675BK160SMT
- moved R2 201.6 mm to (195.5, 46.0), turned to -90 degrees
- moved C3 199.4 mm to (193.4, 46.0), turned to -90 degrees
- moved BOOT1 194.7 mm to (185.2, 48.0)
- moved R17 187.5 mm to (80.0, 66.1), turned to -90 degrees
- moved MODE_B1 185.5 mm to (80.0, 62.5), turned to -90 degrees
- moved R1 183.1 mm to (176.6, 46.7), turned to -90 degrees
- moved C1 180.9 mm to (174.5, 46.7), turned to -90 degrees
- moved R15 178.4 mm to (80.0, 56.2), turned to -90 degrees
- moved RESET1 176.5 mm to (166.7, 48.0), turned to 0 degrees
- moved MODE_A1 176.4 mm to (80.0, 52.6), turned to -90 degrees
- moved R19 16.4 mm to (72.0, 65.8), turned to 0 degrees
- moved MODE_B2 15.2 mm to (70.9, 64.7)
- moved C17 14.1 mm to (285.8, 88.7), turned to 0 degrees
- moved C26 12.3 mm to (72.0, 63.7), turned to 0 degrees
- moved C15 11.4 mm to (297.1, 74.0)
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Connections:
- BOOT1 pad 1: Net-(IC1-IO0) -> Net-(BOOT1-COM_1)
- C1 pad 1: +3.3V -> GND
- C25 pad 1: +3.3V -> GND
- C3 pad 2: Net-(IC1-IO0) -> Net-(BOOT1-COM_1)
- IC1 pad 10: LRCK -> DIN
- IC1 pad 11: DIN -> LRCK
- IC1 pad 12: BCK -> XSMT
- IC1 pad 27: Net-(IC1-IO0) -> Net-(BOOT1-COM_1)
- IC1 pad 9: XSMT -> BCK
- R2 pad 2: Net-(IC1-IO0) -> Net-(BOOT1-COM_1)
Routing:
- net GND: track 0.00 -> 533.3 mm, vias 0 -> 13
- net +3.3V: track 0.00 -> 384.3 mm, vias 0 -> 6
- net +5V: track 0.00 -> 356.6 mm, vias 0 -> 9
- net ROW4: track 0.00 -> 276.6 mm, vias 0 -> 6
- net COL1: track 0.00 -> 255.2 mm, vias 0 -> 2
- net ROW2: track 0.00 -> 239.1 mm, vias 0 -> 5
- net ROW1: track 0.00 -> 230.0 mm, vias 0 -> 4
- net ROW3: track 0.00 -> 228.7 mm, vias 0 -> 6
- net ROW5: track 0.00 -> 225.2 mm, vias 0 -> 6
- net ROW6: track 0.00 -> 222.5 mm, vias 0 -> 5
- net COL2: track 0.00 -> 192.1 mm, vias 0 -> 2
- net Net-(IC1-IO9): track 0.00 -> 169.7 mm, vias 0 -> 3
- net Net-(IC1-IO35): track 0.00 -> 162.7 mm, vias 0 -> 3
- net Net-(IC1-IO3): track 0.00 -> 159.8 mm, vias 0 -> 1
- net Net-(IC1-IO45): track 0.00 -> 157.4 mm, vias 0 -> 2
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- added copper zone on B.Cu, net GND
- added copper zone on F.Cu, net GND
Other:
- board size 293 x 49.5 mm -> 283.9 x 46.2 mm
- board text added: "pcb #5, rev 1 infinite keyboard"
- board text added: "||| _____ /X-X\ \-v-/ /-----\ \-----/ /-------\ \-------/ ~~~~~~~~~"
