File: infinite_keyboard/infinite_keyboard.kicad_sch (KiCad schematic)
At the start: 110 parts, among them IC1 ESP32-S3-WROOM-1-N8, IC2 MIC5504-3.3YM5-TR, IC3 PCM5100APWR, IC4 TPA6130A2RTJR, J1 UJ20-C-H-G-SMT-5-P16-TR, J2 MSD-1-A, J3 SJ-43617-SMT-TR

Commit message: PCB routing
Parts:
- removed C2: 1uF, symbol Device:C
- BOOT1: renamed from BOOT; footprint (none) -> Button_Switch_THT:SW_PUSH_6mm_H4.3mm
- C1, C10, C11, C12, C13, C14, C15, C16, C17, C18, C19, C20, C21, C22, C23, C24, C25, C26, C27, C28, C3, C4, C5, C6, C7, C8, C9: footprint (none) -> Capacitor_SMD:C_0805_2012Metric
- D1, D10, D11, D12, D13, D14, D15, D16, D17, D18, D19, D2, D20, D21, D22, D23, D24, D3, D4, D5, D6, D7, D8, D9: footprint (none) -> Diode_SMD:D_SOD-323F
- IC1: footprint ESP32S3WROOM1N8R2 -> libraries:ESP32S3WROOM1N8R2
- IC2: footprint SOT95P280X145-5N -> libraries:SOT95P280X145-5N
- IC3: footprint SOP65P640X120-20N -> libraries:SOP65P640X120-20N
- IC4: footprint QFN50P400X400X80-21N-D -> libraries:QFN50P400X400X80-21N-D
- J1: footprint UJ20CHGSMT5P16TR -> libraries:UJ20CHGSMT5P16TR
- J2: footprint MSD1A -> libraries:MSD1A
- J3: footprint SJ43617SMTTR -> libraries:SJ43617SMTTR
- MODE_A1: renamed from MODE_A; footprint (none) -> LED_SMD:LED_0805_2012Metric
- MODE_A2: renamed from MODE_A; footprint (none) -> Button_Switch_THT:SW_PUSH_6mm_H4.3mm
- MODE_B1: renamed from MODE_B; footprint (none) -> LED_SMD:LED_0805_2012Metric
- MODE_B2: renamed from MODE_B; footprint (none) -> Button_Switch_THT:SW_PUSH_6mm_H4.3mm
- POWER1: renamed from POWER; footprint (none) -> LED_SMD:LED_0805_2012Metric
- R1, R10, R11, R12, R13, R14, R15, R16, R17, R18, R19, R2, R3, R4, R5, R6, R7, R8, R9: footprint (none) -> Resistor_SMD:R_0805_2012Metric
- RESET1: renamed from RESET; footprint (none) -> Button_Switch_THT:SW_PUSH_6mm_H4.3mm
- RUNNING1: renamed from RUNNING; footprint (none) -> LED_SMD:LED_0805_2012Metric
- SW1, SW10, SW11, SW12, SW13, SW14, SW15, SW16, SW17, SW18, SW19, SW2, SW20, SW21, SW22, SW23, SW24, SW3, SW4, SW5, SW6, SW7, SW8, SW9: footprint (none) -> libraries:CherryMX_1.00u_PCB
Connections:
- net +3.3V: no longer C10.2, C12.1, C12.2, C13.1, C13.2, C14.1, C15.2, C16.2, C17.1, C19.2, C22.2, C23.2, C24.2, C27.2, C28.2, C4.1, C5.1, C6.1, C7.2, C8.2, C9.2, IC1.1 (GND_1), IC1.40 (GND_2), IC1.41 (GND_3), IC1.42 (GND_4), IC1.43 (GND_5), IC1.44 (GND_6), IC1.45 (GND_7), IC1.46 (GND_8), IC1.47 (GND_9), IC1.48 (GND_10), IC1.49 (GND_11), IC2.2 (GND), IC3.10 (DEMP), IC3.11 (FLT), IC3.12 (SCK), IC3.16 (FMT), IC3.18 (LDOO), IC3.19 (DGND), IC3.3 (CPGND), IC3.9 (AGND), IC4.10 (GND_3), IC4.13 (GND_4), IC4.19 (GND_5), IC4.21 (THERMAL_PAD), IC4.3 (GND_1), IC4.9 (GND_2), J1.A1 (GND_1), J1.B1 (GND_2), J2.10 (GND_2), J2.11 (GND_3), J2.12 (GND_4), J2.6 (VSS), J2.9 (GND_1), J3.1 (SLEEVE), MODE_A2.3, MODE_B2.3, R3.1, R4.1, RESET1.3
- net TPA_SCL: no longer R9.1
- net TPA_SDA: now also R9.1
- net at C3.2, IC1.27 (IO0), R2.2: now also BOOT1.1; no longer BOOT1.3
- net at C26.2, IC1.26 (IO45), R19.2: now also MODE_B2.2; no longer MODE_B2.4
- net at C25.2, IC1.28 (IO35), R18.2: now also MODE_A2.2; no longer MODE_A2.4
- net GND: now reaches MODE_A2.1
- net GND: now also BOOT1.2, C10.2, C12.2, C13.2, C14.1, C15.2, C16.2, C17.1, C19.2, C22.2, C23.2, C24.2, C27.2, C28.2, C4.1, C5.1, C6.1, C7.2, C8.2, C9.2, IC1.1 (GND_1), IC1.40 (GND_2), IC1.41 (GND_3), IC1.42 (GND_4), IC1.43 (GND_5), IC1.44 (GND_6), IC1.45 (GND_7), IC1.46 (GND_8), IC1.47 (GND_9), IC1.48 (GND_10), IC1.49 (GND_11), IC2.2 (GND), IC3.10 (DEMP), IC3.11 (FLT), IC3.12 (SCK), IC3.16 (FMT), IC3.19 (DGND), IC3.3 (CPGND), IC3.9 (AGND), IC4.10 (GND_3), IC4.13 (GND_4), IC4.19 (GND_5), IC4.21 (THERMAL_PAD), IC4.3 (GND_1), IC4.9 (GND_2), J1.A1 (GND_1), J1.B1 (GND_2), J2.10 (GND_2), J2.11 (GND_3), J2.12 (GND_4), J2.6 (VSS), J2.9 (GND_1), J3.1 (SLEEVE), MODE_B2.1, R3.1, R4.1, RESET1.3
- net at C22.1, IC4.2 (LEFTINP): no longer C21.2, IC4.5 (RIGHTINM)
- new net: C12.1, C13.1, IC3.18 (LDOO)
- new net: C21.2, IC4.5 (RIGHTINM)
Other:
- moved on the sheet: C22

Commit message: Lots of updates
Parts:
- removed IC2: MIC5504-3.3YM5-TR, libraries:SOT95P280X145-5N, symbol MIC5504-3_3YM5-TR:MIC5504-3.3YM5-TR
- added IC5: AP2112K-3.3TRG1, libraries:SOT95P285X140-5N, symbol AP2112K-3_3TRG1:AP2112K-3.3TRG1
- added R20, R21, R22, R24: 22, Resistor_SMD:R_0805_2012Metric, symbol Device:R_US
- added R23, R25, R26: 10k, Resistor_SMD:R_0805_2012Metric, symbol Device:R_US
- C24, C3: value C -> 1uF
Connections:
- net +3.3V: now also IC5.5 (VOUT), R23.2, R25.2, R26.2; no longer C26.1, C3.1, R13.2
- net +5V: now also R13.2, IC5.1 (VIN)
- net COL1: now also IC1.30 (IO37); no longer IC1.4 (IO4)
- net COL2: now also IC1.31 (IO38); no longer IC1.5 (IO5)
- net COL3: now also IC1.32 (IO39); no longer IC1.6 (IO6)
- net COL4: now also IC1.33 (IO40); no longer IC1.7 (IO7)
- net GND: now also C26.1, C3.1, J3.4 (RING_2), RESET1.1, IC5.2 (GND); no longer RESET1.3
- net ROW1: now also IC1.34 (IO41); no longer IC1.8 (IO15)
- net ROW2: now also IC1.35 (IO42); no longer IC1.9 (IO16)
- net ROW3: now also IC1.36 (RXD0); no longer IC1.10 (IO17)
- net ROW4: now also IC1.37 (TXD0); no longer IC1.11 (IO18)
- net ROW5: now also IC1.38 (IO2); no longer IC1.12 (IO8)
- net ROW6: now also IC1.39 (IO1); no longer IC1.15 (IO3)
- net TPA_SCL: now also IC1.7 (IO7); no longer IC1.30 (IO37)
- net TPA_SDA: now also IC1.8 (IO15); no longer IC1.31 (IO38)
- net at C1.2, IC1.3 (EN), R1.2: now also RESET1.2; no longer RESET1.4
- net BCK: now reaches IC3.13 (BCK)
- net BCK: now also IC1.12 (IO8); no longer IC1.32 (IO39)
- net DIN: now reaches IC3.14 (DIN)
- net DIN: now also IC1.11 (IO18); no longer IC1.33 (IO40)
- net LRCK: now reaches IC3.15 (LRCK)
- net LRCK: now also IC1.10 (IO17); no longer IC1.34 (IO41)
- net XSMT: now reaches IC3.17 (XSMT)
- net XSMT: now also IC1.9 (IO16); no longer IC1.35 (IO42)
- net at MODE_B1.1 (K): now also IC1.15 (IO3); no longer IC1.16 (IO46)
- net at J2.1 (DAT2): now also R26.1
- net at J2.8 (DAT1): now also R25.1
- new net: J2.2 (CD/DAT3), R23.1, R24.1
- new net: IC1.25 (IO48), R24.2
- new net: J2.3 (CMD), R12.1, R22.1
- new net: J2.5 (CLK), R11.1, R21.1
- new net: IC1.22 (IO14), R20.2
- new net: IC1.23 (IO21), R21.2
- new net: IC1.24 (IO47), R22.2
- new net: J2.7 (DAT0), R10.1, R20.1
- new net: IC5.3 (EN), R13.1
Other:
- moved on the sheet: C16, C27, C28

Commit message: Misc changes
Parts:
- removed BOOT1, MODE_A2, MODE_B2, RESET1: SW_Push_Dual, Button_Switch_THT:SW_PUSH_6mm_H4.3mm, symbol Switch:SW_Push_Dual
- added BOOT1, MODE_A2, MODE_B2, RESET1: TS04-66-75-BK-160-SMT, libraries:TS046675BK160SMT, symbol TS04-66-75-BK-160-SMT:TS04-66-75-BK-160-SMT
Connections:
- net +3.3V: no longer C1.1, C25.1
- net BCK: now also IC1.9 (IO16); no longer IC1.12 (IO8)
- net DIN: now also IC1.10 (IO17); no longer IC1.11 (IO18)
- net GND: now also C1.1, C25.1, BOOT1.2 (NO_2), BOOT1.4 (COM_2), MODE_A2.1 (NO_1), MODE_A2.3 (COM_1), MODE_B2.1 (NO_1), MODE_B2.3 (COM_1), RESET1.1 (NO_1)
- net LRCK: now also IC1.11 (IO18); no longer IC1.10 (IO17)
- net XSMT: now also IC1.12 (IO8); no longer IC1.9 (IO16)
- net at C1.2, IC1.3 (EN), R1.2: now also RESET1.2 (NO_2), RESET1.4 (COM_2)
- net at C3.2, IC1.27 (IO0), R2.2: now also BOOT1.1 (NO_1), BOOT1.3 (COM_1)
- net at C26.2, IC1.26 (IO45), R19.2: now also MODE_B2.2 (NO_2), MODE_B2.4 (COM_2)
- net at C25.2, IC1.28 (IO35), R18.2: now also MODE_A2.2 (NO_2), MODE_A2.4 (COM_2)
